Commit message: update with real distances

File: aristos/config/robot.urdf.xacro (robot description, xacro)
@@ -13,5 +13,5 @@
     <parent link="chassis_link" />
     <child link="imu_link" />
-    <origin xyz="0 0 0" rpy="0 0 0" />
+    <origin xyz="0.001 -0.0077 0.28966" rpy="0 0 0" />
   </joint>
   <link name="imu_enu_link"> </link>
@@ -25,5 +25,5 @@
     <parent link="chassis_link" />
     <child link="velodyne" />
-    <origin xyz="0 0 0" rpy="0 0 0" />
+    <origin xyz="0.21 0 0.71" rpy="0 0 ${PI}" />
   </joint>
   <link name="navsat_link"> </link>

Commit message: minor misc

File: aristos/config/robot.urdf.xacro (robot description, xacro)
@@ -21,9 +21,17 @@
     <origin xyz="0 0 0" rpy="0 0 0" />
   </joint>
+  <!-- Domokos -->
+  <!-- <link name="velodyne"> </link>
+  <joint name="velodyne_joint" type="fixed">
+    <parent link="chassis_link" />
+    <child link="velodyne" />
+    <origin xyz="0.21 0 0.71" rpy="0 0 ${PI}" />
+  </joint> -->
+  <!-- Ferrara -->
   <link name="velodyne"> </link>
   <joint name="velodyne_joint" type="fixed">
     <parent link="chassis_link" />
     <child link="velodyne" />
-    <origin xyz="0.21 0 0.71" rpy="0 0 ${PI}" />
+    <origin xyz="0.387 0 0.701" rpy="0.008 0 ${-PI/2.0}" />
   </joint>
   <link name="navsat_link"> </link>

Commit message: livox imu config added

File: aristos/config/robot.urdf.xacro (robot description, xacro)
@@ -29,9 +29,16 @@
   </joint> -->
   <!-- Ferrara -->
+  <!-- <link name="velodyne"> </link>
+  <joint name="velodyne_joint" type="fixed">
+    <parent link="chassis_link" />
+    <child link="velodyne" />
+    <origin xyz="0.387 0 0.701" rpy="0.008 0 ${-PI/2.0}" />
+  </joint> -->
+  <!-- Domokos 2 -->
   <link name="velodyne"> </link>
   <joint name="velodyne_joint" type="fixed">
     <parent link="chassis_link" />
     <child link="velodyne" />
-    <origin xyz="0.387 0 0.701" rpy="0.008 0 ${-PI/2.0}" />
+    <origin xyz="0.387 0 0.701" rpy="-0.077 0 ${-PI/2.0}" />
   </joint>
   <link name="navsat_link"> </link>

Commit message: major: gnss_rmse_heading, onlyRTK, bootstrap filters added +misc

File: aristos/config/robot.urdf.xacro (robot description, xacro)
@@ -29,9 +29,16 @@
   </joint> -->
   <!-- Ferrara -->
+  <!-- <link name="velodyne"> </link>
+  <joint name="velodyne_joint" type="fixed">
+    <parent link="chassis_link" />
+    <child link="velodyne" />
+    <origin xyz="0.387 0 0.701" rpy="0.008 0 ${-PI/2.0}" />
+  </joint> -->
+  <!-- DOMOKOS 2 -->
   <link name="velodyne"> </link>
   <joint name="velodyne_joint" type="fixed">
     <parent link="chassis_link" />
     <child link="velodyne" />
-    <origin xyz="0.387 0 0.701" rpy="0.008 0 ${-PI/2.0}" />
+    <origin xyz="0.387 0 0.631" rpy="0.008 0 ${-PI/2.0}" />
   </joint>
   <link name="navsat_link"> </link>
